File: ptdriver.sch (KiCad schematic (older format))
At the start: 62 parts, among them J1 Power, J10 Heaters, J2 Vout, J3 serial port, J4 3-wire PT100 probe, J5 Conn_01x02, J6 Conn_02x03_Odd_Even, J7 display, J8 3-wire PT100 probe, J9 Vout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

Commit message: Re-arrange and rename things to survive a move from one folder to another
Parts:
- U4, U6: symbol weo:MAX31865_SSOP -> ptdriver-rescue:MAX31865_SSOP-weo
Changed lines of the file:
@@
 	8500 2250 8700 2250
 $Comp
-L weo:MAX31865_SSOP U4
+L ptdriver-rescue:MAX31865_SSOP-weo U4
 U 1 1 6004EB3C
 P 7800 950
@@
 	8800 4350 9000 4350
 $Comp
-L weo:MAX31865_SSOP U6
+L ptdriver-rescue:MAX31865_SSOP-weo U6
 U 1 1 61453592
 P 8100 3050

Commit message: Update picture of board; Fix a couple of windy traces
Parts:
- U4, U6: symbol ptdriver-rescue:MAX31865_SSOP-weo -> ptdriver-rescue:MAX31865_SSOP-weo-ptdriver-rescue
Changed lines of the file:
@@
 	8500 2250 8700 2250
 $Comp
-L ptdriver-rescue:MAX31865_SSOP-weo U4
+L ptdriver-rescue:MAX31865_SSOP-weo-ptdriver-rescue U4
 U 1 1 6004EB3C
 P 7800 950
@@
 	8800 4350 9000 4350
 $Comp
-L ptdriver-rescue:MAX31865_SSOP-weo U6
+L ptdriver-rescue:MAX31865_SSOP-weo-ptdriver-rescue U6
 U 1 1 61453592
 P 8100 3050
